File: Hardware/SparkFun_microSD_Breakout.sch (EAGLE design)
At the start: 7 parts, among them U1 microSD

Commit message: Fixed pin out.
Other:
- note added: "V15"
- note removed: "V01"
Changed lines of the file:
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@@
 <sheet>
 <plain>
-<text x="238.76" y="7.62" size="2.54" layer="94">V01</text>
+<text x="238.76" y="7.62" size="2.54" layer="94">V15</text>
 <text x="148.336" y="7.112" size="2.54" layer="94">Revised by: Patrick Alberts</text>
 </plain>
